Commit message: fix: integrated workspace between real robot and simulation robot, Now can control real robot with imu but not tunning PID and more latency transport.

File: hdt_arm_description/urdf/hdt_arm.urdf (robot description, URDF)
Before this commit: robot hdt_arm, 7 links, 6 joints
Joints:
- joint shoulder_roll_joint: limit lower=-0.1 upper=2.356 effort=35 velocity=2.5 -> lower=-0.1 upper=2.967 effort=35 velocity=2.5
